Commit message: multi_robot simulation experiment

File: URDF import examples/robots_library/aliengo/urdf/aliengo.urdf (robot description, URDF)
Before this commit: robot aliengo_description, 19 links, 18 joints
Links:
- link FL_calf: geometry collision box size=0.25 0.0208 0.016; visual mesh filename=../meshes/calf.stl scale=1 1 1
- link FL_hip: geometry collision cylinder length=0.0418 radius=0.046; visual mesh filename=../meshes/hip.stl scale=1 1 1
- link FL_thigh: geometry collision box size=0.25 0.0374 0.043; visual mesh filename=../meshes/thigh.stl scale=1 1 1
- link FR_calf: geometry collision box size=0.25 0.0208 0.016; visual mesh filename=../meshes/calf.stl scale=1 1 1
- link FR_hip: geometry collision cylinder length=0.0418 radius=0.046; visual mesh filename=../meshes/hip.stl scale=1 1 1
- link FR_thigh: geometry collision box size=0.25 0.0374 0.043; visual mesh filename=../meshes/thigh_mirror.stl scale=1 1 1
- link RL_calf: geometry collision box size=0.25 0.0208 0.016; visual mesh filename=../meshes/calf.stl scale=1 1 1
- link RL_hip: geometry collision cylinder length=0.0418 radius=0.046; visual mesh filename=../meshes/hip.stl scale=1 1 1
- link RL_thigh: geometry collision box size=0.25 0.0374 0.043; visual mesh filename=../meshes/thigh.stl scale=1 1 1
- link RR_calf: geometry collision box size=0.25 0.0208 0.016; visual mesh filename=../meshes/calf.stl scale=1 1 1
- link RR_hip: geometry collision cylinder length=0.0418 radius=0.046; visual mesh filename=../meshes/hip.stl scale=1 1 1
- link RR_thigh: geometry collision box size=0.25 0.0374 0.043; visual mesh filename=../meshes/thigh_mirror.stl scale=1 1 1
- link trunk: geometry collision box size=0.647 0.15 0.112; visual mesh filename=../meshes/trunk.stl scale=1 1 1
Joints:
- joint FL_calf_joint: limit lower=-2.77507351067 upper=-0.645771823238 effort=55 velocity=16 -> lower=-2.77507351067 upper=-0.645771823238 effort=44.4 velocity=40
- joint FL_hip_joint: limit lower=-1.2217304764 upper=1.2217304764 effort=44 velocity=20 -> lower=-1.2217304764 upper=1.2217304764 effort=44.4 velocity=40
- joint FL_thigh_joint: limit effort=44 velocity=20 -> effort=44.4 velocity=40
- joint FR_calf_joint: limit lower=-2.77507351067 upper=-0.645771823238 effort=55 velocity=16 -> lower=-2.77507351067 upper=-0.645771823238 effort=44.4 velocity=40
- joint FR_hip_joint: limit lower=-1.2217304764 upper=1.2217304764 effort=44 velocity=20 -> lower=-1.2217304764 upper=1.2217304764 effort=44.4 velocity=40
- joint FR_thigh_joint: limit effort=44 velocity=20 -> effort=44.4 velocity=40
- joint RL_calf_joint: limit lower=-2.77507351067 upper=-0.645771823238 effort=55 velocity=16 -> lower=-2.77507351067 upper=-0.645771823238 effort=44.4 velocity=40
- joint RL_hip_joint: limit lower=-1.2217304764 upper=1.2217304764 effort=44 velocity=20 -> lower=-1.2217304764 upper=1.2217304764 effort=44.4 velocity=40
- joint RL_thigh_joint: limit effort=44 velocity=20 -> effort=44.4 velocity=40
- joint RR_calf_joint: limit lower=-2.77507351067 upper=-0.645771823238 effort=55 velocity=16 -> lower=-2.77507351067 upper=-0.645771823238 effort=44.4 velocity=40
- joint RR_hip_joint: limit lower=-1.2217304764 upper=1.2217304764 effort=44 velocity=20 -> lower=-1.2217304764 upper=1.2217304764 effort=44.4 velocity=40
- joint RR_thigh_joint: limit effort=44 velocity=20 -> effort=44.4 velocity=40

File: URDF import examples/robots_library/anymal/urdf/anymal_srd.urdf (robot description, URDF)
Before this commit: robot anymal, 23 links, 22 joints
Links:
- link base: mass None -> 16.793507758

File: URDF import examples/robots_library/hyq/urdf/biped.urdf (robot description, URDF)
Before this commit: robot biped, 7 links, 6 joints
Links:
- link L_hipassembly: mass None -> 1.993
- link L_lowerleg: mass None -> 1.993
- link L_upperleg: mass None -> 1.993
- link R_hipassembly: mass None -> 1.993
- link R_upperleg: mass None -> 1.993
- link base: mass None -> 0.5

File: URDF import examples/robots_library/spider/urdf/crab_srd.urdf (robot description, URDF)
Before this commit: robot crab, 32 links, 31 joints
Links:
- link coxa_l1: mass None -> 1.993
- link coxa_l2: mass None -> 1.993
- link coxa_l3: mass None -> 1.993
- link coxa_r1: mass None -> 1.993
- link coxa_r2: mass None -> 1.993
- link coxa_r3: mass None -> 1.993
- link femur_l1: mass None -> 1.993
- link femur_l2: mass None -> 1.993
- link femur_l3: mass None -> 1.993
- link femur_r1: mass None -> 1.993
- link femur_r2: mass None -> 1.993
- link femur_r3: mass None -> 1.993
- link thorax: mass None -> 1.993
- link tibia_l1: mass None -> 1.993
- link tibia_l2: mass None -> 1.993
- link tibia_l3: mass None -> 1.993
- link tibia_r1: mass None -> 1.993
- link tibia_r2: mass None -> 1.993
- link tibia_r3: mass None -> 1.993
